File: Hardware/schematic.sch (EAGLE design)
At the start: 103 parts, among them IC1 XC6220A331MR-G, IC3 BD5229G-TR, J1 SAMACSYS_PARTS_USB4110-GF-A, J2 112A-TAAR-R03_ATTEND, J3 FH34SRJ-24S-0.5SH_99_, J4 QWIIC_RIGHT_ANGLE, Q1 20V/4.2A/52mΩ/1.4W, Q2 SI1308EDL-T1-GE3, Q3 20V/4.2A/52mΩ/1.4W, U1 MCP73831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

Commit message: Resolve Issue 1 2 and add battery cable
Parts:
- D2: value ESP32_WROVER_AVX---SD0805S020S1R0_AVX_SD0805S020S1R0_0_0AVX_SD0805S020S1R0_0_0 -> SD0805S020S1R0
- U3: value BME680 -> BME688
- renumbered R1 to R1_PWRUSB
Other:
- moved on the sheet: U3, U4
